File: STM32_ESP8266_devboard/STM32_ESP8266_devboard.sch (KiCad schematic (older format))
At the start: 16 parts

Commit message: Another commit, not final
Parts:
- added C? (x2): 10pF, symbol Device:C
- added C? (x2): 8pF, symbol Device:C
- added J?: Conn_02x03_Counter_Clockwise, symbol Connector_Generic:Conn_02x03_Counter_Clockwise
- added R? (x3): 10k, symbol Device:R
- added SW?: SW_Push, symbol Switch:SW_Push
- added Y?: 8MHz, symbol Device:Crystal
- added Y?: 32768kHz, symbol Device:Crystal
Connections:
- net +3V3: now also J?.1 (Pin_1), J?.6 (Pin_6), R?.1
- net GND: now also C?.2, C?.2, C?.2, C?.2, J?.3 (Pin_3), J?.4 (Pin_4), SW?.1
- net BOOT1: now reaches U?.20 (PB2)
- net BOOT1: now also R?.2
- net OSC32_IN: now reaches U?.3 (PC14)
- net OSC32_IN: now also C?.1, Y?.1
- net OSC32_OUT: now reaches U?.4 (PC15)
- net OSC32_OUT: now also C?.1, Y?.2
- net BOOT0: now reaches U?.44 (BOOT0)
- net BOOT0: now also R?.1
- net OSC_IN: now reaches U?.5 (PD0)
- net OSC_IN: now also C?.1, Y?.1
- net OSC_OUT: now reaches U?.6 (PD1)
- net OSC_OUT: now also C?.1, Y?.2
- net at U?.7 (NRST): now also R?.2, SW?.2
- new net: J?.2 (Pin_2), R?.2
- new net: J?.5 (Pin_5), R?.1

Commit message: Another commit #2
Parts:
- added C?: 10uF, symbol Device:CP
- added C?: 22uF, symbol Device:CP
- added J?: STM32_PROG, symbol Connector:Conn_01x04_Male
- added J?: ESP_PROG, symbol Connector_Generic:Conn_01x04
- added J?: UART_JMP, symbol Connector_Generic:Conn_02x03_Odd_Even
- added U?: AMS1117-3.3, Package_TO_SOT_SMD:SOT-223-3_TabPin2, symbol Regulator_Linear:AMS1117-3.3
- J?: value Conn_01x03 -> ESP_BOOT
- J?: value Conn_02x03_Counter_Clockwise -> STM32_BOOT_MODE
Connections:
- net +3V3: now also C?.1, J?.1 (Pin_1), J?.1 (Pin_1), U?.2 (VO)
- net GND: now also C?.2, C?.2, J?.4 (Pin_4), J?.4 (Pin_4), U?.1 (GND)
- net STM32_TX: now reaches U?.30 (PA9)
- net STM32_TX: now also J?.1 (Pin_1)
- net STM32_RX: now reaches U?.31 (PA10)
- net STM32_RX: now also J?.2 (Pin_2)
- net SWDIO: now reaches U?.34 (PA13)
- net SWDIO: now also J?.2 (Pin_2)
- net SWCLK: now reaches U?.37 (PA14)
- net SWCLK: now also J?.3 (Pin_3)
- net ESP_RX: now reaches U?.21 (GPIO3/RXD)
- net ESP_RX: now also J?.4 (Pin_4)
- net ESP_TX: now reaches U?.22 (GPIO1/TXD)
- net ESP_TX: now also J?.3 (Pin_3)
- new net +5V: C?.1, U?.3 (VI)
- new net ESP_RX_OUT: J?.2 (Pin_2), J?.6 (Pin_6)
- new net ESP_TX_OUT: J?.3 (Pin_3), J?.5 (Pin_5)
Other:
- moved on the sheet: C?, J?, R?, Y?

Commit message: another one commit
Parts:
- added J?: ESP_GPIO, symbol Connector_Generic:Conn_01x10
- added J?: STM32_GPIO_1, symbol Connector_Generic:Conn_01x13
- added J?: STM32_GPIO_2, symbol Connector_Generic:Conn_01x13
- added J?: STM32_GPIO_3, symbol Connector_Generic:Conn_01x04
- added J?: Conn_01x08, symbol Connector_Generic:Conn_01x08
- added J?: Barrel_Jack, symbol Connector:Barrel_Jack
Connections:
- net +5V: now also J?.1
- net GND: now also J?.10 (Pin_10), J?.13 (Pin_13), J?.13 (Pin_13), J?.2, J?.4 (Pin_4), J?.8 (Pin_8), J?.9 (Pin_9)
- net PA_0: now reaches U?.10 (PA0)
- net PA_0: now also J?.1 (Pin_1)
- net PA_1: now reaches U?.11 (PA1)
- net PA_1: now also J?.2 (Pin_2)
- net PA_2: now reaches U?.12 (PA2)
- net PA_2: now also J?.3 (Pin_3)
- net PA_3: now reaches U?.13 (PA3)
- net PA_3: now also J?.4 (Pin_4)
- net PA_4: now reaches U?.14 (PA4)
- net PA_4: now also J?.5 (Pin_5)
- net PA_5: now reaches U?.15 (PA5)
- net PA_5: now also J?.6 (Pin_6)
- net PA_6: now reaches U?.16 (PA6)
- net PA_6: now also J?.7 (Pin_7)
- net PA_7: now reaches U?.17 (PA7)
- net PA_7: now also J?.8 (Pin_8)
- net PB_0: now reaches U?.18 (PB0)
- net PB_0: now also J?.1 (Pin_1)
- net PB_1: now reaches U?.19 (PB1)
- net PB_1: now also J?.2 (Pin_2)
- net PB_10: now reaches U?.21 (PB10)
- net PB_10: now also J?.10 (Pin_10)
- net PB_11: now reaches U?.22 (PB11)
- net PB_11: now also J?.11 (Pin_11)
- net PB_12: now reaches U?.25 (PB12)
- net PB_12: now also J?.12 (Pin_12)
- net PB_13: now reaches U?.26 (PB13)
- net PB_13: now also J?.1 (Pin_1)
- net PB_14: now reaches U?.27 (PB14)
- net PB_14: now also J?.2 (Pin_2)
- net PB_15: now reaches U?.28 (PB15)
- net PB_15: now also J?.3 (Pin_3)
- net PA_8: now reaches U?.29 (PA8)
- net PA_8: now also J?.9 (Pin_9)
- net PA_11: now reaches U?.32 (PA11)
- net PA_11: now also J?.10 (Pin_10)
- net PA_12: now reaches U?.33 (PA12)
- net PA_12: now also J?.11 (Pin_11)
- net PA_15: now reaches U?.38 (PA15)
- net PA_15: now also J?.12 (Pin_12)
- net PB_3: now reaches U?.39 (PB3)
- net PB_3: now also J?.3 (Pin_3)
- net PB_4: now reaches U?.40 (PB4)
- net PB_4: now also J?.4 (Pin_4)
- net PB_5: now reaches U?.41 (PB5)
- net PB_5: now also J?.5 (Pin_5)
- net PB_6: now reaches U?.42 (PB6)
- net PB_6: now also J?.6 (Pin_6)
- net PB_7: now reaches U?.43 (PB7)
- net PB_7: now also J?.7 (Pin_7)
- net PB_8: now reaches U?.45 (PB8)
- net PB_8: now also J?.8 (Pin_8)
- net PB_9: now reaches U?.46 (PB9)
- net PB_9: now also J?.9 (Pin_9)
- net ESP_MISO: now reaches U?.10 (MISO)
- net ESP_MISO: now also J?.5 (Pin_5)
- net ESP_SDD2: now reaches U?.11 (GPIO9)
- net ESP_SDD2: now also J?.2 (Pin_2)
- net ESP_SDD3: now reaches U?.12 (GPIO10)
- net ESP_SDD3: now also J?.3 (Pin_3)
- net ESP_MOSI: now reaches U?.13 (MOSI)
- net ESP_MOSI: now also J?.6 (Pin_6)
- net ESP_SCLK: now reaches U?.14 (SCLK)
- net ESP_SCLK: now also J?.7 (Pin_7)
- net ESP_D8: now reaches R?.2, U?.16 (GPIO15)
- net ESP_D8: now also J?.8 (Pin_8)
- net ESP_D2: now reaches U?.19 (GPIO4)
- net ESP_D2: now also J?.3 (Pin_3)
- net ESP_ADC: now reaches U?.2 (ADC)
- net ESP_ADC: now also J?.1 (Pin_1)
- net ESP_D1: now reaches U?.20 (GPIO5)
- net ESP_D1: now also J?.2 (Pin_2)
- net ESP_D0: now reaches U?.4 (GPIO16)
- net ESP_D0: now also J?.1 (Pin_1)
- net ESP_D5: now reaches U?.5 (GPIO14)
- net ESP_D5: now also J?.5 (Pin_5)
- net ESP_D6: now reaches U?.6 (GPIO12)
- net ESP_D6: now also J?.6 (Pin_6)
- net ESP_D7: now reaches U?.7 (GPIO13)
- net ESP_D7: now also J?.7 (Pin_7)
- net ESP_CSO: now reaches U?.9 (CS0)
- net ESP_CSO: now also J?.4 (Pin_4)
- net GPIO_0 renamed ESP_D3
- net ESP_D3: now also J?.4 (Pin_4)
- no-connect marks 0 -> 1
Other:
- moved on the sheet: R?

Commit message: another one commit#3
Parts:
- added D1: ON_LED(R), symbol Device:LED
- added D?: STM32_LED(B), symbol Device:LED
- added D?: ESP_LED(G), symbol Device:LED
- added J8: EXTERNAL_3,3V, symbol Connector_Generic:Conn_01x02
- added R4, R? (x2): 200, symbol Device:R
- gave numbers to parts that had none: 39
Connections:
- net +3V3: now also J8.1 (Pin_1), R4.1
- net ESP_D3: now also R?.1
- net GND: now also D1.1 (K), D?.1 (K), D?.1 (K), J8.2 (Pin_2)
- net PA_1: now also R?.1
- net STM32_RX: now also J2.1 (Pin_1); no longer J2.2 (Pin_2)
- net STM32_TX: now also J2.2 (Pin_2); no longer J2.1 (Pin_1)
- new net: D1.2 (A), R4.2
- new net: D?.2 (A), R?.2 (x2)

Commit message: Final principal scheme
Parts:
- gave numbers to parts that had none: 4
Changed lines of the file:
@@
 PA_1
 $Comp
-L Device:R R?
+L Device:R R10
 U 1 1 5F4ABBD3
 P 7050 3800
-F 0 "R?" H 7120 3846 50  0000 L CNN
+F 0 "R10" H 7120 3846 50  0000 L CNN
 F 1 "200" H 7120 3755 50  0000 L CNN
 F 2 "" V 6980 3800 50  0001 C CNN
@@
 $EndComp
 $Comp
-L Device:LED D?
+L Device:LED D2
 U 1 1 5F4ABC5B
 P 7050 4200
-F 0 "D?" V 7088 4082 50  0000 R CNN
+F 0 "D2" V 7088 4082 50  0000 R CNN
 F 1 "STM32_LED(B)" V 6997 4082 50  0000 R CNN
 F 2 "" H 7050 4200 50  0001 C CNN
@@
 $EndComp
 $Comp
-L power:GND #PWR?
+L power:GND #PWR0140
 U 1 1 5F4ABCDD
 P 7050 4450
-F 0 "#PWR?" H 7050 4200 50  0001 C CNN
+F 0 "#PWR0140" H 7050 4200 50  0001 C CNN
 F 1 "GND" H 7055 4277 50  0000 C CNN
 F 2 "" H 7050 4450 50  0001 C CNN
@@
 GPIO_0
 $Comp
-L Device:R R?
+L Device:R R11
 U 1 1 5F4C4E32
 P 8000 3800
-F 0 "R?" H 8070 3846 50  0000 L CNN
+F 0 "R11" H 8070 3846 50  0000 L CNN
 F 1 "200" H 8070 3755 50  0000 L CNN
 F 2 "" V 7930 3800 50  0001 C CNN
@@
 $EndComp
 $Comp
-L Device:LED D?
+L Device:LED D3
 U 1 1 5F4C4ECC
 P 8000 4200
-F 0 "D?" V 8038 4082 50  0000 R CNN
+F 0 "D3" V 8038 4082 50  0000 R CNN
 F 1 "ESP_LED(G)" V 7947 4082 50  0000 R CNN
 F 2 "" H 8000 4200 50  0001 C CNN
@@
 	8000 3950 8000 4050
 $Comp
-L power:GND #PWR?
+L power:GND #PWR0141
 U 1 1 5F4D1892
 P 8000 4450
-F 0 "#PWR?" H 8000 4200 50  0001 C CNN
+F 0 "#PWR0141" H 8000 4200 50  0001 C CNN
 F 1 "GND" H 8005 4277 50  0000 C CNN
 F 2 "" H 8000 4450 50  0001 C CNN
@@
 Wire Wire Line
 	8000 4350 8000 4450
+$Comp
+L power:PWR_FLAG #FLG0101
+U 1 1 5F49347A
+P 4000 4950
+F 0 "#FLG0101" H 4000 5025 50  0001 C CNN
+F 1 "PWR_FLAG" H 4000 5124 50  0000 C CNN
+F 2 "" H 4000 4950 50  0001 C CNN
+F 3 "~" H 4000 4950 50  0001 C CNN
+	1    4000 4950
+	1    0    0    -1
+$EndComp
+$Comp
+L power:PWR_FLAG #FLG0102
+U 1 1 5F493572
+P 4500 4950
+F 0 "#FLG0102" H 4500 5025 50  0001 C CNN
+F 1 "PWR_FLAG" H 4500 5124 50  0000 C CNN
+F 2 "" H 4500 4950 50  0001 C CNN
+F 3 "~" H 4500 4950 50  0001 C CNN
+	1    4500 4950
+	1    0    0    -1
+$EndComp
+$Comp
+L power:PWR_FLAG #FLG0103
+U 1 1 5F4935D9
+P 3550 4950
+F 0 "#FLG0103" H 3550 5025 50  0001 C CNN
+F 1 "PWR_FLAG" H 3550 5124 50  0000 C CNN
+F 2 "" H 3550 4950 50  0001 C CNN
+F 3 "~" H 3550 4950 50  0001 C CNN
+	1    3550 4950
+	1    0    0    -1
+$EndComp
+$Comp
+L power:GND #PWR0142
+U 1 1 5F493640
+P 3550 5100
+F 0 "#PWR0142" H 3550 4850 50  0001 C CNN
+F 1 "GND" H 3555 4927 50  0000 C CNN
+F 2 "" H 3550 5100 50  0001 C CNN
+F 3 "" H 3550 5100 50  0001 C CNN
+	1    3550 5100
+	1    0    0    -1
+$EndComp
+$Comp
+L power:+5V #PWR0143
+U 1 1 5F4936A7
+P 4000 5100
+F 0 "#PWR0143" H 4000 4950 50  0001 C CNN
+F 1 "+5V" H 4015 5273 50  0000 C CNN
+F 2 "" H 4000 5100 50  0001 C CNN
+F 3 "" H 4000 5100 50  0001 C CNN
+	1    4000 5100
+	-1   0    0    1
+$EndComp
+$Comp
+L power:+3.3V #PWR0144
+U 1 1 5F49376A
+P 4500 5100
+F 0 "#PWR0144" H 4500 4950 50  0001 C CNN
+F 1 "+3.3V" H 4515 5273 50  0000 C CNN
+F 2 "" H 4500 5100 50  0001 C CNN
+F 3 "" H 4500 5100 50  0001 C CNN
+	1    4500 5100
+	-1   0    0    1
+$EndComp
+Wire Wire Line
+	3550 4950 3550 5100
+Wire Wire Line
+	4000 4950 4000 5100
+Wire Wire Line
+	4500 4950 4500 5100
 $EndSCHEMATC

Commit message: Begin PCB
Parts:
- C1, C10, C13, C2, C3, C4, C5, C6, C7, C8, C9: footprint (none) -> Capacitor_SMD:C_0805_2012Metric
- C11: footprint (none) -> Capacitor_THT:CP_Radial_D5.0mm_P2.50mm
- C12: footprint (none) -> Capacitor_THT:CP_Radial_D5.0mm_P2.00mm
- D1, D2, D3: footprint (none) -> LED_SMD:LED_0805_2012Metric
- J1, J12, J3: footprint (none) -> Connector_PinHeader_2.54mm:PinHeader_1x04_P2.54mm_Vertical
- J10: footprint (none) -> Connector_PinHeader_2.54mm:PinHeader_1x10_P2.54mm_Vertical
- J11: footprint (none) -> Connector_PinHeader_2.54mm:PinHeader_1x03_P2.54mm_Vertical
- J2, J5: footprint (none) -> Connector_PinHeader_2.54mm:PinHeader_2x03_P2.54mm_Vertical
- J4, J6: footprint (none) -> Connector_PinHeader_2.54mm:PinHeader_1x13_P2.54mm_Vertical
- J7: footprint (none) -> Connector_BarrelJack:BarrelJack_Horizontal
- J8: footprint (none) -> Connector_PinHeader_2.54mm:PinHeader_1x02_P2.54mm_Vertical
- J9: value Conn_01x08 -> ESP_GPIO2; footprint (none) -> Connector_PinHeader_2.54mm:PinHeader_1x08_P2.54mm_Vertical
- R1, R10, R11, R2, R3, R4, R5, R6, R7, R8, R9: footprint (none) -> Resistor_SMD:R_0805_2012Metric
- SW1, SW2: footprint (none) -> Button_Switch_THT:SW_PUSH_6mm
- Y1, Y2: footprint (none) -> Crystal:Crystal_HC52-8mm_Vertical

Commit message: Another one commit, not final
Parts:
- Y2: footprint Crystal:Crystal_HC52-8mm_Vertical -> Crystal:Crystal_DS26_D2.0mm_L6.0mm_Horizontal_1EP_style1
Changed lines of the file:
@@
 F 0 "Y2" H 2650 7218 50  0000 C CNN
 F 1 "32768kHz" H 2650 7127 50  0000 C CNN
-F 2 "Crystal:Crystal_HC52-8mm_Vertical" H 2650 6950 50  0001 C CNN
+F 2 "Crystal:Crystal_DS26_D2.0mm_L6.0mm_Horizontal_1EP_style1" H 2650 6950 50  0001 C CNN
 F 3 "~" H 2650 6950 50  0001 C CNN
 	1    2650 6950

Commit message: Все хуйня, разводи плату по новой
Connections:
- net +3V3: now also J5.2 (Pin_2); no longer J5.6 (Pin_6)
- net ESP_CSO: now also J9.7 (Pin_7); no longer J9.4 (Pin_4)
- net ESP_MISO: now also J9.6 (Pin_6); no longer J9.5 (Pin_5)
- net ESP_MOSI: now also J9.3 (Pin_3); no longer J9.6 (Pin_6)
- net ESP_RX_OUT: now also J2.5 (Pin_5); no longer J2.6 (Pin_6)
- net ESP_SCLK: now also J9.2 (Pin_2); no longer J9.7 (Pin_7)
- net ESP_SDD2: now also J9.5 (Pin_5); no longer J9.2 (Pin_2)
- net ESP_SDD3: now also J9.4 (Pin_4); no longer J9.3 (Pin_3)
- net ESP_TX_OUT: now also J2.6 (Pin_6); no longer J2.5 (Pin_5)
- net GND: now also J5.5 (Pin_5), J5.6 (Pin_6); no longer J5.3 (Pin_3), J5.4 (Pin_4)
- net PB_0: now also J4.12 (Pin_12); no longer J4.1 (Pin_1)
- net PB_1: now also J4.11 (Pin_11); no longer J4.2 (Pin_2)
- net PB_11: now also J4.9 (Pin_9); no longer J4.11 (Pin_11)
- net PB_12: now also J4.8 (Pin_8); no longer J4.12 (Pin_12)
- net PB_13: now also J4.7 (Pin_7); no longer J3.1 (Pin_1)
- net PB_14: now also J4.6 (Pin_6); no longer J3.2 (Pin_2)
- net PB_15: now also J4.5 (Pin_5); no longer J3.3 (Pin_3)
- net PB_5: now also J4.2 (Pin_2); no longer J4.5 (Pin_5)
- net PB_6: now also J4.1 (Pin_1); no longer J4.6 (Pin_6)
- net PB_7: now also J3.3 (Pin_3); no longer J4.7 (Pin_7)
- net PB_8: now also J3.1 (Pin_1); no longer J4.8 (Pin_8)
- net PB_9: now also J3.2 (Pin_2); no longer J4.9 (Pin_9)
- net SWCLK: now also J1.2 (Pin_2); no longer J1.3 (Pin_3)
- net SWDIO: now also J1.3 (Pin_3); no longer J1.2 (Pin_2)
- net at R2.2: now also J5.3 (Pin_3); no longer J5.2 (Pin_2)
- net at R3.1: now also J5.4 (Pin_4); no longer J5.5 (Pin_5)
Other:
- moved on the sheet: R2, R3
Changed lines of the file:
@@
 Text Label 2050 2600 2    50   ~ 0
 BOOT1
-Text Label 5050 7150 2    50   ~ 0
+Text Label 5050 7250 2    50   ~ 0
 BOOT0
 $Comp
@@
 L Device:R R3
 U 1 1 5F478C8B
-P 6300 7150
-F 0 "R3" H 6370 7196 50  0000 L CNN
-F 1 "10k" H 6370 7105 50  0000 L CNN
-F 2 "Resistor_SMD:R_0805_2012Metric" V 6230 7150 50  0001 C CNN
-F 3 "~" H 6300 7150 50  0001 C CNN
-	1    6300 7150
+P 6300 7250
+F 0 "R3" H 6370 7296 50  0000 L CNN
+F 1 "10k" H 6370 7205 50  0000 L CNN
+F 2 "Resistor_SMD:R_0805_2012Metric" V 6230 7250 50  0001 C CNN
+F 3 "~" H 6300 7250 50  0001 C CNN
+	1    6300 7250
 	0    -1   -1   0
 $EndComp
@@
 L Device:R R2
 U 1 1 5F478E8B
-P 5300 7150
-F 0 "R2" H 5370 7196 50  0000 L CNN
-F 1 "10k" H 5370 7105 50  0000 L CNN
-F 2 "Resistor_SMD:R_0805_2012Metric" V 5230 7150 50  0001 C CNN
-F 3 "~" H 5300 7150 50  0001 C CNN
-	1    5300 7150
+P 5300 7250
+F 0 "R2" H 5370 7296 50  0000 L CNN
+F 1 "10k" H 5370 7205 50  0000 L CNN
+F 2 "Resistor_SMD:R_0805_2012Metric" V 5230 7250 50  0001 C CNN
+F 3 "~" H 5300 7250 50  0001 C CNN
+	1    5300 7250
 	0    -1   -1   0
 $EndComp
-Text Label 6600 7150 0    50   ~ 0
+Text Label 6600 7250 0    50   ~ 0
 BOOT1
 Wire Wire Line
-	6050 7150 6150 7150
-Wire Wire Line
-	6450 7150 6600 7150
-Wire Wire Line
-	5050 7150 5150 7150
-Wire Wire Line
-	5450 7150 5550 7150
+	6050 7250 6150 7250
+Wire Wire Line
+	6450 7250 6600 7250
+Wire Wire Line
+	5050 7250 5150 7250
+Wire Wire Line
+	5450 7250 5550 7250
 $Comp
 L power:+3.3V #PWR0118
@@
 	1    0    0    -1
 $EndComp
-$Comp
-L power:+3.3V #PWR0119
-U 1 1 5F484C75
-P 6050 6750
-F 0 "#PWR0119" H 6050 6600 50  0001 C CNN
-F 1 "+3.3V" H 6065 6923 50  0000 C CNN
-F 2 "" H 6050 6750 50  0001 C CNN
-F 3 "" H 6050 6750 50  0001 C CNN
-	1    6050 6750
-	1    0    0    -1
-$EndComp
-$Comp
-L power:GND #PWR0120
-U 1 1 5F484CD4
-P 5550 7400
-F 0 "#PWR0120" H 5550 7150 50  0001 C CNN
-F 1 "GND" H 5555 7227 50  0000 C CNN
-F 2 "" H 5550 7400 50  0001 C CNN
-F 3 "" H 5550 7400 50  0001 C CNN
-	1    5550 7400
-	1    0    0    -1
-$EndComp
-$Comp
-L power:GND #PWR0121
-U 1 1 5F484D1C
-P 6050 7400
-F 0 "#PWR0121" H 6050 7150 50  0001 C CNN
-F 1 "GND" H 6055 7227 50  0000 C CNN
-F 2 "" H 6050 7400 50  0001 C CNN
-F 3 "" H 6050 7400 50  0001 C CNN
-	1    6050 7400
-	1    0    0    -1
-$EndComp
-Wire Wire Line
-	5550 7250 5550 7400
-Wire Wire Line
-	6050 7250 6050 7400
-Wire Wire Line
-	6050 6750 6050 7050
 Wire Wire Line
 	5550 6750 5550 7050
@@
 	1    0    0    -1
 $EndComp
+Text Label 4050 7200 0    50   ~ 0
+SWDIO
 Text Label 4050 7100 0    50   ~ 0
-SWDIO
-Text Label 4050 7200 0    50   ~ 0
 SWCLK
 $Comp
@@
 Text Label 3900 6000 2    50   ~ 0
 ESP_TX
-Text Label 3900 6100 2    50   ~ 0
+Text Label 4400 6100 0    50   ~ 0
 ESP_TX_OUT
 Text Label 3900 5900 2    50   ~ 0
 STM32_RX
-Text Label 4400 6100 0    50   ~ 0
+Text Label 3900 6100 2    50   ~ 0
 ESP_RX_OUT
 Text Label 4400 6000 0    50   ~ 0
@@
 Text Label 2050 3900 2    50   ~ 0
 PB_15
-Text Label 4400 2300 2    50   ~ 0
+Text Label 4400 3400 2    50   ~ 0
 PB_0
-Text Label 4400 2400 2    50   ~ 0
+Text Label 4400 3300 2    50   ~ 0
 PB_1
 Text Label 4400 2500 2    50   ~ 0
@@
 Text Label 4400 2600 2    50   ~ 0
 PB_4
-Text Label 4400 2700 2    50   ~ 0
+Text Label 4400 2400 2    50   ~ 0
 PB_5
-Text Label 4400 2800 2    50   ~ 0
+Text Label 4400 2300 2    50   ~ 0
 PB_6
-Text Label 4400 2900 2    50   ~ 0
+Text Label 4400 1450 2    50   ~ 0
 PB_7
-Text Label 4400 3000 2    50   ~ 0
+Text Label 4400 1250 2    50   ~ 0
 PB_8
-Text Label 4400 3100 2    50   ~ 0
+Text Label 4400 1350 2    50   ~ 0
 PB_9
 Text Label 4400 3200 2    50   ~ 0
 PB_10
-Text Label 4400 3300 2    50   ~ 0
+Text Label 4400 3100 2    50   ~ 0
 PB_11
-Text Label 4400 3400 2    50   ~ 0
+Text Label 4400 3000 2    50   ~ 0
 PB_12
 $Comp
@@
 Wire Wire Line
 	4350 1550 4400 1550
-Text Label 4400 1250 2    50   ~ 0
+Text Label 4400 2900 2    50   ~ 0
 PB_13
-Text Label 4400 1350 2    50   ~ 0
+Text Label 4400 2800 2    50   ~ 0
 PB_14
-Text Label 4400 1450 2    50   ~ 0
+Text Label 4400 2700 2    50   ~ 0
 PB_15
 Text Label 8750 2700 2    50   ~ 0
@@
 Text Label 8000 5100 2    50   ~ 0
 ESP_ADC
+Text Label 8000 5700 2    50   ~ 0
+ESP_CSO
+Text Label 8000 5500 2    50   ~ 0
+ESP_SDD2
 Text Label 8000 5400 2    50   ~ 0
-ESP_CSO
+ESP_SDD3
+Text Label 8000 5600 2    50   ~ 0
+ESP_MISO
+Text Label 8000 5300 2    50   ~ 0
+ESP_MOSI
 Text Label 8000 5200 2    50   ~ 0
-ESP_SDD2
-Text Label 8000 5300 2    50   ~ 0
-ESP_SDD3
-Text Label 8000 5500 2    50   ~ 0
-ESP_MISO
-Text Label 8000 5600 2    50   ~ 0
-ESP_MOSI
-Text Label 8000 5700 2    50   ~ 0
 ESP_SCLK
 $Comp
@@
 Wire Wire Line
 	4500 4950 4500 5100
+Wire Wire Line
+	5550 7150 5550 7050
+Connection ~ 5550 7050
+$Comp
+L power:GND #PWR0119
+U 1 1 5F5BED15
+P 6050 6700
+F 0 "#PWR0119" H 6050 6450 50  0001 C CNN
+F 1 "GND" H 6055 6527 50  0000 C CNN
+F 2 "" H 6050 6700 50  0001 C CNN
+F 3 "" H 6050 6700 50  0001 C CNN
+	1    6050 6700
+	-1   0    0    1
+$EndComp
+Wire Wire Line
+	6050 7150 6050 7050
+Wire Wire Line
+	6050 7050 6050 6700
+Connection ~ 6050 7050
 $EndSCHEMATC
