File: STM32_ESP8266_devboard/STM32_ESP8266_devboard.sch (KiCad schematic (older format))
At the start: 46 parts, among them J1 STM32_PROG, J10 ESP_GPIO, J11 ESP_BOOT, J12 ESP_PROG, J2 UART_JMP, J3 STM32_GPIO_3, J4 STM32_GPIO_2, J5 STM32_BOOT_MODE, J6 STM32_GPIO_1, J7 Barrel_Jack, J8 EXTERNAL_3,3V, J9 ESP_GPIO2, SW1 SW_Push, SW2 SW_Push, U1 STM32F103C8Tx, U2 AMS1117-3.3, U3 ESP-12E, Y1 8MHz, Y2 32768kHz

Commit message: Final version, add logos
Connections:
- net PA_0: now also R10.1
- net PA_1: no longer R10.1
Changed lines of the file:
@@
 	6300 4450 6300 4350
 Text Label 7050 3450 0    50   ~ 0
-PA_1
+PA_0
 $Comp
 L Device:R R10

Commit message: Pre-final pcb
Connections:
- net ESP_RX: now also J2.3 (Pin_3); no longer J2.4 (Pin_4)
- net ESP_TX: now also J2.4 (Pin_4); no longer J2.3 (Pin_3)
Changed lines of the file:
@@
 Text Label 4400 5900 0    50   ~ 0
 STM32_TX
-Text Label 3900 6000 2    50   ~ 0
+Text Label 4400 6000 0    50   ~ 0
 ESP_TX
 Text Label 4400 6100 0    50   ~ 0
@@
 Text Label 3900 6100 2    50   ~ 0
 ESP_RX_OUT
-Text Label 4400 6000 0    50   ~ 0
+Text Label 3900 6000 2    50   ~ 0
 ESP_RX
 $Comp
