File: STM32_ESP8266_devboard/STM32_ESP8266_devboard.kicad_pcb (KiCad board)
At the start: 2 copper layers, 90 x 90 mm, 46 parts, among them J1 STM32_PROG, J10 ESP_GPIO, J11 ESP_BOOT, J12 ESP_PROG, J2 UART_JMP, J3 STM32_GPIO_3, J4 STM32_GPIO_2, J5 STM32_BOOT_MODE, J6 STM32_GPIO_1, J7 Barrel_Jack, J8 EXTERNAL_3,3V, J9 ESP_GPIO2, SW1 SW_Push, SW2 SW_Push, U1 STM32F103C8Tx, U2 AMS1117-3.3, U3 ESP-12E, Y1 8MHz, Y2 32768kHz

Commit message: Another commit
Parts:
- added REF**: MountingHole_3.2mm_M3_Pad, MountingHole:MountingHole_3.2mm_M3_Pad, F.Cu at (125.1, 134.0)
- added REF**: MountingHole_3.2mm_M3_Pad, MountingHole:MountingHole_3.2mm_M3_Pad, F.Cu at (205.7, 134.0)
- added REF**: MountingHole_3.2mm_M3_Pad, MountingHole:MountingHole_3.2mm_M3_Pad, F.Cu at (205.7, 54.0)
- added REF**: MountingHole_3.2mm_M3_Pad, MountingHole:MountingHole_3.2mm_M3_Pad, F.Cu at (125.1, 54.0)
- moved SW1 243.9 mm to (87.0, 181.6)
- moved SW2 228.1 mm to (97.2, 181.6)
- moved R8 185.6 mm to (263.2, 97.2)
- moved R5 183.7 mm to (268.3, 94.6)
- moved R9 180.8 mm to (268.3, 91.4)
- moved R11 180.0 mm to (268.3, 88.3)
- moved R7 179.0 mm to (263.2, 93.3)
- moved C10 176.6 mm to (249.3, 98.4)
- moved R6 176.2 mm to (268.3, 84.5)
- moved R4 175.0 mm to (263.2, 88.3)
- moved C9 173.8 mm to (244.8, 97.2), turned to 180 degrees
- moved R10 173.4 mm to (268.3, 81.3)
- moved R2 172.1 mm to (263.2, 82.5)
- moved D1 171.7 mm to (28.3, 121.3)
- moved C8 171.4 mm to (244.8, 92.7)
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Routing:
- net +3V3: track 0.00 -> 90.9 mm
- net GND: track 0.00 -> 72.8 mm
- net +5V: track 0.00 -> 17.6 mm

Commit message: Another day another commit
Parts:
- moved J10 177.5 mm to (207.3, 63.5)
- moved D3 176.0 mm to (200.2, 90.3), turned to 90 degrees
- moved J11 146.9 mm to (190.5, 94.0), turned to 90 degrees
- moved C6 109.8 mm to (142.2, 113.7), turned to 270 degrees
- moved C10 107.9 mm to (141.7, 107.6), turned to 90 degrees
- moved C1 103.4 mm to (148.8, 104.6), turned to 180 degrees
- moved C8 101.6 mm to (144.3, 107.6), turned to 90 degrees
- moved R5 100.8 mm to (171.2, 67.6), turned to 270 degrees
- moved C5 99.5 mm to (156.5, 119.9)
- moved R7 93.8 mm to (171.2, 75.3), turned to 270 degrees
- moved C3 90.6 mm to (160.0, 108.1), turned to 90 degrees
- moved R11 71.7 mm to (196.6, 90.3), turned to 270 degrees
- moved R8 70.5 mm to (193.0, 90.3), turned to 90 degrees
- moved R9 65.3 mm to (203.1, 87.4), turned to 180 degrees
- moved U1 20.7 mm to (152.1, 112.3)
Routing:
- net GND: track 72.8 -> 161.1 mm
- net /ESP_D7: track 0.00 -> 55.2 mm, vias 0 -> 1
- net /ESP_D6: track 0.00 -> 53.6 mm, vias 0 -> 1
- net /ESP_D5: track 0.00 -> 52.5 mm, vias 0 -> 1
- net /ESP_D3: track 0.00 -> 48.4 mm, vias 0 -> 2
- net /ESP_D0: track 0.00 -> 47.8 mm, vias 0 -> 1
- net /ESP_D8: track 0.00 -> 35.9 mm, vias 0 -> 1
- net Net-(R7-Pad2): track 0.00 -> 35.6 mm, vias 0 -> 2
- net +3V3: track 90.9 -> 113.8 mm, vias 0 -> 1
- net /ESP_D1: track 0.00 -> 17.4 mm
- net /ESP_D2: track 0.00 -> 17.3 mm
- net Net-(R5-Pad1): track 0.00 -> 9.78 mm
- net Net-(D3-Pad2): track 0.00 -> 4.63 mm
- net Net-(J11-Pad2): track 0.00 -> 2.70 mm

Commit message: Another one commit, not final
Parts:
- Y2: footprint Crystal:Crystal_HC52-8mm_Vertical -> Crystal:Crystal_DS26_D2.0mm_L6.0mm_Horizontal_1EP_style1
- moved Y1 140.5 mm to (131.2, 124.1)
- moved J6 130.5 mm to (134.6, 135.1)
- moved C2 129.1 mm to (131.1, 128.4), turned to 270 degrees
- moved C4 119.0 mm to (135.0, 128.5), turned to 270 degrees
- moved Y2 111.0 mm to (147.5, 92.1), turned to 180 degrees
- moved C9 102.0 mm to (143.0, 92.1)
- moved C7 98.9 mm to (150.3, 92.1)
- moved C6 3.71 mm to (142.2, 117.4)
Routing:
- net GND: track 161.1 -> 396.7 mm, vias 0 -> 8
- net /OSC32_OUT: track 0.00 -> 36.8 mm
- net /OSC32_IN: track 0.00 -> 36.7 mm
- net /PA_0: track 0.00 -> 29.4 mm
- net /OSC_IN: track 0.00 -> 29.2 mm
- net /PA_1: track 0.00 -> 26.9 mm
- net /OSC_OUT: track 0.00 -> 26.9 mm
- net /PA_2: track 0.00 -> 24.7 mm
- net /PA_3: track 0.00 -> 21.4 mm
- net /PA_4: track 0.00 -> 20.6 mm
- net /PA_5: track 0.00 -> 19.7 mm
- net /PA_6: track 0.00 -> 18.9 mm
- net /PA_7: track 0.00 -> 18.9 mm
- net +3V3: track 113.8 -> 126.9 mm, vias 1 -> 0
- net +5V: track 17.6 -> 16.1 mm

Commit message: Все хуйня, разводи плату по новой
Parts:
- added ESP_BOOT(J11): ESP_BOOT, Connector_PinHeader_2.54mm:PinHeader_1x03_P2.54mm_Vertical, F.Cu at (190.5, 94.0)
- moved J4 206.9 mm to (199.4, 135.1), turned to 270 degrees
- moved J9 188.5 mm to (207.4, 94.9)
- moved J5 187.0 mm to (232.6, 102.8)
- moved SW2 164.3 mm to (225.4, 78.9)
- moved J1 132.6 mm to (160.1, 103.5), turned to 90 degrees
- moved J3 103.4 mm to (123.2, 105.2), turned to 0 degrees
- moved J12 96.7 mm to (122.2, 90.1), turned to 180 degrees
- moved J2 92.3 mm to (145.6, 75.5), turned to 180 degrees
- moved R3 62.6 mm to (219.3, 116.9)
- moved J11 60.7 mm to (165.0, 149.1), turned to 0 degrees
- moved R2 57.6 mm to (221.1, 121.8)
Connections:
- J1 pad 2: /SWDIO -> /SWCLK
- J1 pad 3: /SWCLK -> /SWDIO
- J2 pad 5: /ESP_TX_OUT -> /ESP_RX_OUT
- J2 pad 6: /ESP_RX_OUT -> /ESP_TX_OUT
- J3 pad 1: /PB_13 -> /PB_8
- J3 pad 2: /PB_14 -> /PB_9
- J3 pad 3: /PB_15 -> /PB_7
- J4 pad 1: /PB_0 -> /PB_6
- J4 pad 11: /PB_11 -> /PB_1
- J4 pad 12: /PB_12 -> /PB_0
- J4 pad 2: /PB_1 -> /PB_5
- J4 pad 5: /PB_5 -> /PB_15
- J4 pad 6: /PB_6 -> /PB_14
- J4 pad 7: /PB_7 -> /PB_13
- J4 pad 8: /PB_8 -> /PB_12
- J4 pad 9: /PB_9 -> /PB_11
- J5 pad 2: Net-(J5-Pad2) -> +3V3
- J5 pad 3: GND -> Net-(J5-Pad3)
- J5 pad 4: GND -> Net-(J5-Pad4)
- J5 pad 5: Net-(J5-Pad5) -> GND
- J5 pad 6: +3V3 -> GND
- J9 pad 2: /ESP_SDD2 -> /ESP_SCLK
- J9 pad 3: /ESP_SDD3 -> /ESP_MOSI
- J9 pad 4: /ESP_CSO -> /ESP_SDD3
- J9 pad 5: /ESP_MISO -> /ESP_SDD2
- J9 pad 6: /ESP_MOSI -> /ESP_MISO
- J9 pad 7: /ESP_SCLK -> /ESP_CSO
- R2 pad 2: Net-(J5-Pad2) -> Net-(J5-Pad3)
- R3 pad 1: Net-(J5-Pad5) -> Net-(J5-Pad4)
Routing:
- net GND: track 396.7 -> 0.00 mm, vias 8 -> 0
- net +3V3: track 126.9 -> 0.00 mm
- net /ESP_D7: track 55.2 -> 0.00 mm, vias 1 -> 0
- net /ESP_D6: track 53.6 -> 0.00 mm, vias 1 -> 0
- net /ESP_D5: track 52.5 -> 0.00 mm, vias 1 -> 0
- net /ESP_D3: track 48.4 -> 0.00 mm, vias 2 -> 0
- net /ESP_D0: track 47.8 -> 0.00 mm, vias 1 -> 0
- net /OSC32_OUT: track 36.8 -> 0.00 mm
- net /OSC32_IN: track 36.7 -> 0.00 mm
- net /ESP_D8: track 35.9 -> 0.00 mm, vias 1 -> 0
- net Net-(R7-Pad2): track 35.6 -> 0.00 mm, vias 2 -> 0
- net /PA_0: track 29.4 -> 0.00 mm
- net /OSC_IN: track 29.2 -> 0.00 mm
- net /PA_1: track 26.9 -> 0.00 mm
- net /OSC_OUT: track 26.9 -> 0.00 mm
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Other:
- board text added: "0"
- board text added: "1"
- board text added: "D0"
- board text added: "D1"
- board text added: "D2"
- board text added: "D3"
- board text added: "D5"
- board text added: "D6"
- board text added: "D7"
- board text added: "D8"
- board text added: "GND"

Commit message: another commit
Parts:
- moved J3 120.9 mm to (28.4, 30.2)
- moved ESP_BOOT(J11) 115.2 mm to (75.3, 96.2)
- moved J1 101.2 mm to (85.6, 35.0)
- moved J12 85.8 mm to (208.0, 91.0), turned to 0 degrees
- moved J9 85.5 mm to (122.0, 97.4), turned to 180 degrees
- moved C7 67.6 mm to (87.2, 67.8)
- moved Y2 67.6 mm to (84.4, 67.8)
- moved C9 67.6 mm to (79.9, 67.8)
- moved C6 55.7 mm to (97.0, 84.9)
- moved J2 55.0 mm to (197.6, 93.6), turned to 270 degrees
- moved C3 29.3 mm to (130.8, 109.7)
- moved C13 28.4 mm to (213.7, 88.4)
- moved D3 28.4 mm to (228.2, 94.9)
- moved R11 28.4 mm to (224.6, 94.9)
- moved R8 28.4 mm to (221.0, 94.9)
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Routing:
- net +3V3: track 0.00 -> 120.2 mm, vias 0 -> 1
- net GND: track 0.00 -> 92.2 mm, vias 0 -> 1
- net /ESP_ADC: track 0.00 -> 82.1 mm, vias 0 -> 2
- net /ESP_SCLK: track 0.00 -> 71.2 mm, vias 0 -> 1
- net /ESP_MOSI: track 0.00 -> 68.2 mm, vias 0 -> 1
- net /ESP_SDD3: track 0.00 -> 65.4 mm, vias 0 -> 1
- net /ESP_D0: track 0.00 -> 63.9 mm, vias 0 -> 1
- net /ESP_SDD2: track 0.00 -> 62.4 mm, vias 0 -> 1
- net /ESP_MISO: track 0.00 -> 61.0 mm, vias 0 -> 1
- net /ESP_CSO: track 0.00 -> 55.6 mm, vias 0 -> 2
- net /ESP_D5: track 0.00 -> 55.3 mm, vias 0 -> 1
- net /ESP_D6: track 0.00 -> 55.3 mm, vias 0 -> 1
- net /ESP_D7: track 0.00 -> 52.5 mm, vias 0 -> 1
- net /ESP_RX: track 0.00 -> 48.4 mm
- net /ESP_TX: track 0.00 -> 47.3 mm
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Other:
- board text removed: "D0"
- board text removed: "D1"
- board text removed: "D2"
- board text removed: "D3"
- board text removed: "D5"
- board text removed: "D6"
- board text removed: "D7"
- board text removed: "D8"
- board text removed: "GND"

Commit message: Another one
Parts:
- removed J11: ESP_BOOT, Connector_PinHeader_2.54mm:PinHeader_1x03_P2.54mm_Vertical
- moved ESP_BOOT(J11) 124.6 mm to (199.2, 82.8), turned to 180 degrees
- moved J1 113.6 mm to (185.0, 90.0), turned to 0 degrees
- moved R6 111.8 mm to (160.2, 55.9)
- moved SW2 75.4 mm to (150.3, 71.2), turned to 90 degrees
- moved J5 62.0 mm to (170.8, 97.4), turned to 90 degrees
- moved C10 61.1 mm to (81.9, 117.9)
- moved C3 61.1 mm to (69.9, 115.1)
- moved C1 61.1 mm to (77.3, 113.7)
- moved C5 61.1 mm to (72.6, 119.3)
- moved C8 61.1 mm to (65.6, 118.4)
- moved C6 56.5 mm to (153.1, 78.1)
- moved R2 52.0 mm to (173.4, 100.9), turned to 90 degrees
- moved C13 47.5 mm to (168.0, 75.6)
- moved R3 46.4 mm to (175.7, 100.9), turned to 270 degrees
- moved R8 33.3 mm to (200.3, 69.0)
Routing:
- net GND: track 92.2 -> 239.5 mm, vias 1 -> 4
- net /BOOT1: track 0.00 -> 49.5 mm, vias 0 -> 2
- net +3V3: track 120.2 -> 167.4 mm
- net /SWDIO: track 0.00 -> 27.5 mm, vias 0 -> 1
- net /SWCLK: track 0.00 -> 27.1 mm, vias 0 -> 2
- net Net-(R6-Pad2): track 0.00 -> 20.0 mm, vias 0 -> 1
- net Net-(J11-Pad2): track 0.00 -> 13.0 mm
- net /BOOT0: track 0.00 -> 8.54 mm
- net /ESP_D3: track 25.5 -> 33.2 mm
- net Net-(J5-Pad4): track 0.00 -> 6.08 mm
- net Net-(J5-Pad3): track 0.00 -> 2.62 mm
- net /ESP_MISO: track 61.0 -> 59.1 mm, vias 1 -> 2
- net /ESP_SCLK: track 71.2 -> 72.9 mm, vias 1 -> 2
- net /ESP_MOSI: track 68.2 -> 69.2 mm, vias 1 -> 2
- net /ESP_ADC: track 82.1 -> 82.7 mm
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Other:
- board text added: "3,3V"
- board text added: "BOOT0"
- board text added: "BOOT1"
- board text added: "GND"
- board text added: "SWCLK"
- board text added: "SWDIO"

Commit message: Final version, add logos
Parts:
- moved D1 130.2 mm to (146.5, 66.8), turned to 180 degrees
- moved J3 126.3 mm to (124.0, 112.8), turned to 180 degrees
- moved D2 124.1 mm to (152.2, 120.9)
- moved R4 119.2 mm to (146.5, 64.0), turned to 180 degrees
- moved R10 118.7 mm to (156.4, 120.9), turned to 180 degrees
- moved C8 112.6 mm to (178.1, 122.8)
- moved C3 111.3 mm to (181.1, 110.0)
- moved J8 111.1 mm to (140.5, 64.0)
- moved SW1 104.6 mm to (139.5, 91.1)
- moved R1 99.6 mm to (165.4, 97.1), turned to 180 degrees
- moved C5 96.8 mm to (168.5, 106.6), turned to 270 degrees
- moved C10 88.1 mm to (168.5, 101.3), turned to 180 degrees
- moved C1 84.0 mm to (161.2, 117.1), turned to 270 degrees
- moved C9 80.5 mm to (152.8, 101.9), turned to 90 degrees
- moved Y2 80.5 mm to (156.8, 102.8)
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- renumbered D3 to ESP_LED(D3)
Connections:
- R10 pad 1: /PA_1 -> /PA_0
Routing:
- net GND: track 239.5 -> 509.2 mm, vias 4 -> 16
- net +3V3: track 167.4 -> 302.4 mm, vias 1 -> 6
- net /PB_7: track 0.00 -> 79.5 mm, vias 0 -> 4
- net /PA_15: track 0.00 -> 74.9 mm, vias 0 -> 3
- net /PB_6: track 0.00 -> 68.4 mm, vias 0 -> 7
- net /PA_11: track 0.00 -> 68.3 mm, vias 0 -> 3
- net /PA_12: track 0.00 -> 67.6 mm, vias 0 -> 3
- net /PA_8: track 0.00 -> 65.4 mm, vias 0 -> 3
- net /PB_5: track 0.00 -> 64.8 mm, vias 0 -> 6
- net /PB_8: track 0.00 -> 60.2 mm, vias 0 -> 5
- net /PB_9: track 0.00 -> 56.3 mm, vias 0 -> 4
- net /PB_4: track 0.00 -> 54.1 mm, vias 0 -> 2
- net /PA_0: track 0.00 -> 50.5 mm
- net /PB_3: track 0.00 -> 49.0 mm, vias 0 -> 1
- net /PA_1: track 0.00 -> 45.4 mm
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- added copper zone on B.Cu, net GND
Other:
- board text added: "+"

Commit message: Pre-final pcb
Parts:
- moved R11 2.60 mm to (202.6, 70.3)
- renumbered ESP_BOOT(J11) to ESP_BOOT
Connections:
- J2 pad 3: /ESP_TX -> /ESP_RX
- J2 pad 4: /ESP_RX -> /ESP_TX
Routing:
- net /ESP_RX: track 48.4 -> 42.4 mm
- net /ESP_D3: track 35.1 -> 34.5 mm
- net Net-(D3-Pad2): track 17.5 -> 16.9 mm
Other:
- board text added: "."
- board text added: "3.3V"
- board text added: "D0"
- board text added: "D1"
- board text added: "D2"
- board text added: "D3"
- board text added: "D5"
- board text added: "D6"
- board text added: "D7"
- board text added: "D8"
- board text added: "ESP"
- board text added: "ESP-UART"
- board text added: "ESP_ADC"
- board text added: "ESP_CSO"
- board text added: "ESP_MISO"
- board text added: "ESP_MOSI"
- board text added: "ESP_RST"
- board text added: "ESP_SCLK"
- board text added: "ESP_SDD2"
- board text added: "ESP_SDD3"
- board text added: "PA0"
- board text added: "PA1"
- board text added: "PA11"
- board text added: "PA12"
- board text added: "PA15"
- board text added: "PA2"
- board text added: "PA3"
- board text added: "PA4"
- board text added: "PA5"
- board text added: "PA6"
- board text added: "PA7"
- board text added: "PA8"
- board text added: "PB0"
- board text added: "PB1"
- board text added: "PB10"
- board text added: "PB11"
- board text added: "PB12"
- board text added: "PB13"
- board text added: "PB14"
- board text added: "PB15"
- board text added: "PB3"
- board text added: "PB4"
- board text added: "PB5"
- board text added: "PB6"
- board text added: "PB7"
- board text added: "PB8"
- board text added: "PB9"
- board text added: "RX"
- board text added: "STM"
- board text added: "STM_RST"
- board text added: "TX"
